File: PI PowerSyppy Board/PI_PowerSupply_Board/PI_PowerSupply_Board.kicad_sch (KiCad schematic)
At the start: 19 parts, among them IC1 MIC841HYC5-TR, J1 S4B-PH-K-S_LF__SN_, J2 USB4216-03-A, J3 USB4216-03-A

Commit message: PCB Design
Parts:
- added H1, H2, H3, H4: MountingHole_Pad, MountingHole:MountingHole_2.7mm_M2.5_DIN965_Pad_TopBottom, symbol Mechanical:MountingHole_Pad
- added J4: M20-7832046, BassinaLib_Connectors:RHDR40W65P254_2X20_5120X504X850P, symbol BassinaLib_Connectors:M20-7832046
- added LED1, LED2: GREEN LED, BassinaLib_LEDs:LEDM168X80N, symbol BassinaLib_LEDs:APHD1608LZGCK
- added LED3: RED LED, BassinaLib_LEDs:LEDM168X80N, symbol BassinaLib_LEDs:APHD1608LSURCK
- added R13, R14: 2k 0.1%, Resistor_SMD:R_0603_1608Metric, symbol Device:R
- added R15: 10k 0.1%, Resistor_SMD:R_0603_1608Metric, symbol Device:R
Connections:
- net +VDC: now also R15.1
- net GND: now also H1.1, H2.1, H3.1, H4.1, LED1.1 (K), LED2.1 (K), LED3.1 (K)
- net +5V renamed +5V_A
- net +5V_A: now also R14.1; no longer J3.A4 (VBUS_1), J3.B4 (VBUS_2), R6.1, R8.1
- new net: LED1.2 (A), R13.2
- new net: LED3.2 (A), R15.2
- new net: LED2.2 (A), R14.2
- new net +5V_B: J3.A4 (VBUS_1), J3.B4 (VBUS_2), R13.1, R6.1, R8.1
- no-connect marks 13 -> 53
Other:
- note added: "Mounting holes"
